File: Hardware/KiCAD/Main/ESP8266-WebRadio.kicad_pcb (KiCad board)
At the start: 2 copper layers, 52.5 x 36.6 mm, 49 parts, among them K1 AUDIO, K2 POWER, K3 EARPHONES, P1 UART, P2 PROG, U1 LM1117-3.3, U2 LM1117-1.8, U3 23LCV1024, U4 ESP8266_ESP-12, U5 NE5532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

Commit message: Added pullups in schematic and PCB
Parts:
- added R11: 10k, SM0805, F.Cu at (47.8, 48.3)
- added R12: 10k, SM0805, B.Cu at (54.2, 42.6)
- added R13: 10k, SM0805, B.Cu at (58.0, 38.2)
- moved P2 0.51 mm to (59.1, 45.6), turned to 0 degrees
Connections:
- U4 pad 11: (no net) -> N-0000017
Routing:
- net N-0000017: track 0.00 -> 23.1 mm, vias 0 -> 1
- net N-0000029: track 51.4 -> 65.5 mm
- net +3.3V: track 130.3 -> 140.7 mm
- net N-0000031: track 28.4 -> 30.1 mm
